File: Hardware/BeeperAddOn/BeeperAddOn.kicad_pcb (KiCad board)
At the start: 2 copper layers, 12.8 x 20.1 mm, 6 parts, among them J1 Conn_01x03_Socket, Q1 BSS138

Commit message: buzzer
Parts:
- added C2: C, Capacitor_SMD:C_0603_1608Metric, F.Cu at (147.7, 106.2)
- moved C1 1.62 mm to (149.6, 106.2)
- moved Q1 1.55 mm to (152.2, 105.6)
Routing:
- net GND: track 6.70 -> 0.00 mm
- net +3.3V: track 10.4 -> 12.0 mm
- net Net-(Q1-G): track 2.31 -> 3.54 mm
- net Net-(BZ1--): track 8.78 -> 8.17 mm
- added copper zone on F.Cu, net GND

Commit message: Buzzer
Parts:
- moved BZ1 59.3 mm to (108.6, 68.3)
- moved C2 59.3 mm to (110.3, 60.2)
- moved Q1 59.3 mm to (114.7, 59.7)
- moved C1 59.3 mm to (112.1, 60.2)
- moved J1 59.3 mm to (107.7, 61.3)
- moved R1 59.3 mm to (113.0, 56.4)
- moved R2 59.3 mm to (110.5, 57.1)
Changed lines of the file:
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@@
 		(legacy_teardrops no)
 	)
-	(paper "A4")
+	(paper "A5")
 	(layers
 		(0 "F.Cu" signal)
@@
 		(allow_soldermask_bridges_in_footprints no)
 		(pcbplotparams
-			(layerselection 0x00010fc_ffffffff)
+			(layerselection 0x0000000_7fffffff)
 			(plot_on_all_layers_selection 0x0000000_00000000)
 			(disableapertmacros no)
@@
 			(sketchpadsonfab no)
 			(subtractmaskfromsilk no)
-			(outputformat 1)
-			(mirror no)
-			(drillshape 1)
+			(outputformat 4)
+			(mirror yes)
+			(drillshape 2)
 			(scaleselection 1)
 			(outputdirectory "")
@@
 	(footprint "Buzzer_Beeper:Buzzer_12x9.5RM7.6"
 		(layer "F.Cu")
-		(at 146.08 114.28)
+		(at 108.63 68.33)
 		(descr "Generic Buzzer, D12mm height 9.5mm with RM7.6mm")
 		(tags "buzzer")
@@
 	(footprint "Capacitor_SMD:C_0603_1608Metric"
 		(layer "F.Cu")
-		(at 147.71 106.2 90)
+		(at 110.26 60.25 90)
 		(descr "Capacitor SMD 0603 (1608 Metric), square (rectangular) end terminal, IPC_7351 nominal, (Body size source: IPC-SM-782 page 76, https://www.pcb-3d.com/wordpress/wp-content/uploads/ipc-sm-782a_amendment_1_and_2.pdf), generated with kicad-footprint-generator")
 		(tags "capacitor")
 		(property "Reference" "C2"
-			(at 0 -1.43 270)
+			(at 0 -1.43 -90)
 			(layer "F.SilkS")
 			(effects
@@
 		)
 		(property "Value" "C"
-			(at 0 1.43 270)
+			(at 0 1.43 -90)
 			(layer "F.Fab")
 			(effects
@@
 		)
 		(fp_text user "${REFERENCE}"
-			(at 0 0 270)
+			(at 0 0 -90)
 			(layer "F.Fab")
 			(effects
@@
 	(footprint "Resistor_SMD:R_0603_1608Metric"
 		(layer "F.Cu")
-		(at 150.415 102.32)
+		(at 112.965 56.37)
 		(descr "Resistor SMD 0603 (1608 Metric), square (rectangular) end terminal, IPC_7351 nominal, (Body size source: IPC-SM-782 page 72, https://www.pcb-3d.com/wordpress/wp-content/uploads/ipc-sm-782a_amendment_1_and_2.pdf), generated with kicad-footprint-generator")
 		(tags "resistor")
@@
 	(footprint "Capacitor_SMD:C_0603_1608Metric"
 		(layer "F.Cu")
-		(at 149.56 106.195 90)
+		(at 112.11 60.245 90)
 		(descr "Capacitor SMD 0603 (1608 Metric), square (rectangular) end terminal, IPC_7351 nominal, (Body size source: IPC-SM-782 page 76, https://www.pcb-3d.com/wordpress/wp-content/uploads/ipc-sm-782a_amendment_1_and_2.pdf), generated with kicad-footprint-generator")
 		(tags "capacitor")
@@
 	(footprint "Resistor_SMD:R_0603_1608Metric"
 		(layer "F.Cu")
-		(at 147.92 103.07 90)
+		(at 110.47 57.12 90)
 		(descr "Resistor SMD 0603 (1608 Metric), square (rectangular) end terminal, IPC_7351 nominal, (Body size source: IPC-SM-782 page 72, https://www.pcb-3d.com/wordpress/wp-content/uploads/ipc-sm-782a_amendment_1_and_2.pdf), generated with kicad-footprint-generator")
 		(tags "resistor")
@@
 	(footprint "Package_TO_SOT_SMD:SOT-23-3"
 		(layer "F.Cu")
-		(at 152.15 105.61 -90)
+		(at 114.7 59.66 -90)
 		(descr "SOT, 3 Pin (https://www.jedec.org/sites/default/files/docs/Mo-178D.PDF inferred 3-pin variant), generated with kicad-footprint-generator ipc_gullwing_generator.py")
 		(tags "SOT TO_SOT_SMD")
@@
 	(footprint "Connector_PinSocket_2.54mm:PinSocket_1x03_P2.54mm_Vertical"
 		(layer "B.Cu")
-		(at 145.12 107.27)
+		(at 107.67 61.32)
 		(descr "Through hole straight socket strip, 1x03, 2.54mm pitch, single row (from Kicad 4.0.7), script generated")
 		(tags "Through hole socket strip THT 1x03 2.54mm single row")
@@
 	)
 	(gr_rect
-		(start 143.41 100.38)
-		(end 156.17 120.46)
+		(start 105.8 54.3)
+		(end 118.9 74.7)
+		(stroke
+			(width 0.2)
+			(type default)
+		)
+		(fill none)
+		(layer "F.Cu")
+	)
+	(gr_rect
+		(start 105.96 54.43)
+		(end 118.72 74.51)
 		(stroke
 			(width 0.1)
@@
 	)
 	(segment
-		(start 145.41 106.98)
-		(end 149.55 106.98)
+		(start 107.96 61.03)
+		(end 112.1 61.03)
 		(width 0.75)
 		(layer "F.Cu")
@@
 	)
 	(segment
-		(start 145.12 113.32)
-		(end 146.08 114.28)
+		(start 107.67 67.37)
+		(end 108.63 68.33)
 		(width 1)
 		(layer "F.Cu")
@@
 	)
 	(segment
-		(start 149.55 106.98)
-		(end 149.56 106.97)
+		(start 112.1 61.03)
+		(end 112.11 61.02)
 		(width 0.75)
 		(layer "F.Cu")
@@
 	)
 	(segment
-		(start 145.12 107.27)
-		(end 145.41 106.98)
+		(start 107.67 61.32)
+		(end 107.96 61.03)
 		(width 0.75)
 		(layer "F.Cu")
@@
 	)
 	(segment
-		(start 145.12 107.27)
-		(end 145.12 113.32)
+		(start 107.67 61.32)
+		(end 107.67 67.37)
 		(width 1)
 		(layer "F.Cu")
@@
 	)
 	(segment
-		(start 152.15 112.75)
-		(end 153.68 114.28)
+		(start 114.7 66.8)
+		(end 116.23 68.33)
 		(width 1)
 		(layer "F.Cu")
@@
 	)
 	(segment
-		(start 152.15 106.7475)
-		(end 152.15 112.75)
+		(start 114.7 60.7975)
+		(end 114.7 66.8)
 		(width 1)
 		(layer "F.Cu")
@@
 	)
 	(segment
-		(start 153.1 103.13)
-		(end 153.1 104.4725)
+		(start 115.65 57.18)
+		(end 115.65 58.5225)
 		(width 0.75)
 		(layer "F.Cu")
@@
 	)
 	(segment
-		(start 152.29 102.32)
-		(end 153.1 103.13)
+		(start 114.84 56.37)
+		(end 115.65 57.18)
 		(width 0.75)
 		(layer "F.Cu")
@@
 	)
 	(segment
-		(start 151.24 102.32)
-		(end 152.29 102.32)
+		(start 113.79 56.37)
+		(end 114.84 56.37)
 		(width 0.75)
 		(layer "F.Cu")
@@
 	)
 	(segment
-		(start 149.515 102.245)
-		(end 149.59 102.32)
+		(start 112.065 56.295)
+		(end 112.14 56.37)
 		(width 0.75)
 		(layer "F.Cu")
@@
 	)
 	(segment
-		(start 147.92 102.245)
-		(end 149.515 102.245)
+		(start 110.47 56.295)
+		(end 112.065 56.295)
 		(width 0.75)
 		(layer "F.Cu")
@@
 	)
 	(segment
-		(start 147.865 102.19)
-		(end 147.92 102.245)
+		(start 110.415 56.24)
+		(end 110.47 56.295)
 		(width 0.75)
 		(layer "F.Cu")
@@
 	)
 	(segment
-		(start 145.12 102.19)
-		(end 147.865 102.19)
+		(start 107.67 56.24)
+		(end 110.415 56.24)
 		(width 0.75)
 		(layer "F.Cu")
@@
 		(polygon
 			(pts
-				(xy 143.9 103.5) (xy 151.5 103.5) (xy 151.5 105.1) (xy 150.5 105.9) (xy 143.9 105.9)
-			)
-		)
+				(xy 106.45 57.55) (xy 114.05 57.55) (xy 114.05 59.15) (xy 113.05 59.95) (xy 106.45 59.95)
+			)
+		)
