File: Hardware/PreciPSLoadFront V3/PreciPSLoadFront.kicad_sch (KiCad schematic)
At the start: 55 parts, among them J1 Ch1, J2 Ch2, J3 Fan, J4 Display, J5 KeyPad, J6 12Vin, J7 ExtPw, J9 Ext, Q1 DMG6968, SW1 SW_Push, SW10 RotaryEncoder_Switch, SW11 SW_Push, SW2 SW_Push, SW3 SW_Push, SW4 SW_Push, SW5 SW_Push, SW6 SW_Push, SW7 SW_Push, SW8 SW_Push, SW9 SW_Push, U2 Teensy4.1, U3 LM317_TO-220

Commit message: IoT
Other:
- moved on the sheet: J7
Changed lines of the file:
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@@
 	(generator "eeschema")
 	(generator_version "8.0")
-	(paper "A3")
+	(paper "A4")
 	(junction
 		(at 85.09 172.085)
@@
 	(symbol
 		(lib_id "Connector:Conn_01x03_Pin")
-		(at 211.455 167.005 270)
+		(at 241.3 140.97 270)
 		(unit 1)
 		(exclude_from_sim no)
@@
 		(fields_autoplaced yes)
 		(property "Reference" "J7"
-			(at 211.455 162.56 90)
+			(at 241.3 136.525 90)
 			(effects
 				(font
@@
 		)
 		(property "Value" "ExtPw"
-			(at 211.455 165.1 90)
+			(at 241.3 139.065 90)
 			(effects
 				(font
@@
 		)
 		(property "Footprint" "Connector_JST:JST_XH_B3B-XH-A_1x03_P2.50mm_Vertical"
-			(at 211.455 167.005 0)
+			(at 241.3 140.97 0)
 			(effects
 				(font
@@
 		)
 		(property "Datasheet" "~"
-			(at 211.455 167.005 0)
+			(at 241.3 140.97 0)
 			(effects
 				(font
@@
 		)
 		(property "Description" "Generic connector, single row, 01x03, script generated"
-			(at 211.455 167.005 0)
+			(at 241.3 140.97 0)
 			(effects
 				(font
@@
 	(symbol
 		(lib_id "power:+5V")
-		(at 208.915 172.085 180)
+		(at 238.76 146.05 180)
 		(unit 1)
 		(exclude_from_sim no)
@@
 		(dnp no)
 		(property "Reference" "#PWR033"
-			(at 208.915 168.275 0)
+			(at 238.76 142.24 0)
 			(effects
 				(font
@@
 		)
 		(property "Value" "+5V"
-			(at 207.645 177.8 0)
+			(at 237.49 151.765 0)
 			(effects
 				(font
@@
 		)
 		(property "Footprint" ""
-			(at 208.915 172.085 0)
+			(at 238.76 146.05 0)
 			(effects
 				(font
@@
 		)
 		(property "Datasheet" ""
-			(at 208.915 172.085 0)
+			(at 238.76 146.05 0)
 			(effects
 				(font
@@
 		)
 		(property "Description" "Power symbol creates a global label with name \"+5V\""
-			(at 208.915 172.085 0)
+			(at 238.76 146.05 0)
 			(effects
 				(font
@@
 	(symbol
 		(lib_id "power:GND")
-		(at 213.995 172.085 0)
+		(at 243.84 146.05 0)
 		(unit 1)
 		(exclude_from_sim no)
@@
 		(fields_autoplaced yes)
 		(property "Reference" "#PWR03"
-			(at 213.995 178.435 0)
+			(at 243.84 152.4 0)
 			(effects
 				(font
@@
 		)
 		(property "Value" "GND"
-			(at 213.995 176.53 0)
+			(at 243.84 150.495 0)
 			(effects
 				(font
@@
 		)
 		(property "Footprint" ""
-			(at 213.995 172.085 0)
+			(at 243.84 146.05 0)
 			(effects
 				(font
@@
 		)
 		(property "Datasheet" ""
-			(at 213.995 172.085 0)
+			(at 243.84 146.05 0)
 			(effects
 				(font
@@
 		)
 		(property "Description" "Power symbol creates a global label with name \"GND\" , ground"
-			(at 213.995 172.085 0)
+			(at 243.84 146.05 0)
 			(effects
 				(font
@@
 	(symbol
 		(lib_id "power:+3V3")
-		(at 211.455 172.085 180)
+		(at 241.3 146.05 180)
 		(unit 1)
 		(exclude_from_sim no)
@@
 		(dnp no)
 		(property "Reference" "#PWR045"
-			(at 211.455 168.275 0)
+			(at 241.3 142.24 0)
 			(effects
 				(font
@@
 		)
 		(property "Value" "+3V3"
-			(at 212.09 177.8 0)
+			(at 241.935 151.765 0)
 			(effects
 				(font
@@
 		)
 		(property "Footprint" ""
-			(at 211.455 172.085 0)
+			(at 241.3 146.05 0)
 			(effects
 				(font
@@
 		)
 		(property "Datasheet" ""
-			(at 211.455 172.085 0)
+			(at 241.3 146.05 0)
 			(effects
 				(font
@@
 		)
 		(property "Description" "Power symbol creates a global label with name \"+3V3\""
-			(at 211.455 172.085 0)
+			(at 241.3 146.05 0)
 			(effects
 				(font
@@
 		(dnp no)
 		(property "Reference" "J4"
-			(at 24.765 12.065 0)
+			(at 18.796 28.448 0)
 			(effects
 				(font
@@
 		)
 		(property "Value" "Display"
-			(at 24.765 14.605 0)
+			(at 18.796 30.988 0)
 			(effects
 				(font
