File: Hardware/PrezisoinPowerSupply V12/PrezisoinPowerSupply.kicad_sch (KiCad schematic)
At the start: 155 parts, among them J1 Supply, J2 Conn_01x03_Pin, J3 Conn_02x05_Odd_Even, J4 LEDs, J5 Sense, J6 Output, K1 EE2-5NU, Q1 IRFP240, Q2 IRFP9240, Q4 IRFP9240, Q5 MMBT3904, Q6 MMBT3904, Q7 MMBT3904, Q8 MMBT3904, Q9 IRFP240, U10 OPA4189, U11 OPA4189, U12 OPA189, U16 ATtiny3227-M, U19 TLV9301xDBV, U2 DG469, U21 ADS1219, U3 ADA4522, U4 CPC1017N, U5 ISO7763FDBQ, U7 DAC8564C/D, U8 MCP9700Ax-ETT, U9 MCP9700Ax-ETT

Commit message: IoT
Other:
- note removed: "Vss, Vdd low offset"
- note removed: "Vss, Vdd low offset matched R"
- note removed: "Vss, Vdd no prezision"
- company: (none) -> Jannik Schreiber
- title: (none) -> PSLoad
Changed lines of the file:
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@@
 	(generator_version "8.0")
 	(paper "A2")
+	(title_block
+		(title "PSLoad")
+		(company "Jannik Schreiber")
+	)
 	(junction
 		(at 195.58 196.215)
@@
 		)
 	)
-	(text "Vss, Vdd\nlow offset\n"
-		(exclude_from_sim no)
-		(at 314.96 82.55 0)
-		(effects
-			(font
-				(size 1.27 1.27)
-			)
-		)
-	)
 	(text "any IO"
 		(exclude_from_sim no)
@@
 	(text "LSB 0,000 000 596 ..."
 		(exclude_from_sim no)
-		(at 154.94 190.5 0)
+		(at 84.582 218.186 0)
 		(effects
 			(font
@@
 		)
 	)
-	(text "Vss, Vdd\nno prezision\n"
-		(exclude_from_sim no)
-		(at 300.355 150.495 0)
-		(effects
-			(font
-				(size 1.27 1.27)
-			)
-		)
-	)
 	(text "any IO"
 		(exclude_from_sim no)
@@
 	(text "-5A +5A\n2,5V 0V"
 		(exclude_from_sim no)
-		(at 114.3 155.575 0)
+		(at 117.094 168.148 0)
 		(effects
 			(font
@@
 	(text "V mes \nLSB 100uV\nmax 25, 000 0 V"
 		(exclude_from_sim no)
-		(at 146.685 46.355 0)
+		(at 149.86 59.309 0)
 		(effects
 			(font
@@
 	(text "V set\nLSB 1 mV\nmax 25 V"
 		(exclude_from_sim no)
-		(at 146.685 55.88 0)
+		(at 149.86 68.834 0)
 		(effects
 			(font
@@
 	(text "Gain x10\nin +- 0,25V\nout +- 2,5V"
 		(exclude_from_sim no)
-		(at 371.475 137.16 0)
+		(at 371.348 137.922 0)
 		(effects
 			(font
@@
 		)
 	)
-	(text "Vss, Vdd\nlow offset\nmatched R\n"
-		(exclude_from_sim no)
-		(at 278.13 65.405 0)
-		(effects
-			(font
-				(size 1.27 1.27)
-			)
-		)
-	)
 	(text "I mes\nLSB 10uA\nmax 5,000 00"
 		(exclude_from_sim no)
-		(at 169.545 46.355 0)
+		(at 172.72 59.309 0)
 		(effects
 			(font
@@
 	(text "I set\nLSB 1 mA (100 uA)\nmax 5 A"
 		(exclude_from_sim no)
-		(at 169.545 55.88 0)
+		(at 172.72 68.834 0)
 		(effects
 			(font
