File: Hardware/Modul/PrezisoinPowerSupply 2_2/PrezisoinPowerSupply.kicad_sch (KiCad schematic)
At the start: 163 parts, among them J1 Supply, J2 Conn_01x03_Pin, J3 Conn_02x05_Odd_Even, J4 LEDs, J5 Sense, J6 Output, K1 EE2-5NU, Q1 IRFP240, Q2 IRFP9240, Q4 IRFP9240, Q5 MMBT3904, Q6 MMBT3904, Q7 MMBT3904, Q8 MMBT3904, Q9 IRFP240, U10 OPA4189, U11 OPA4189, U12 OPA189, U16 ATtiny3227-M, U19 TLV9301xDBV, U2 DG469, U21 ADS1219, U3 ADA4522, U4 CPC1017N, U5 ISO7763FDBQ, U7 DAC8564C/D, U8 MCP9700Ax-ETT, U9 MCP9700Ax-ETT

Commit message: improove gnd
Parts:
- removed D9: SS10PH10, Package_TO_SOT_SMD:TO-277A, symbol Device:D_AAK
- added NT4: Tie, NetTie:NetTie-2_SMD_Pad2.0mm, symbol Device:NetTie_2
Connections:
- net GND: now also NT4.2; no longer Q2.2 (D), Q4.2 (D), R51.4
- new net GNDPWR: NT4.1, Q2.2 (D), Q4.2 (D), R51.4

Commit message: work hardware
Parts:
- added C19, C39: 100n, Capacitor_SMD:C_0603_1608Metric, symbol Device:C
- added D9: 1N4148WS, Diode_SMD:D_SOD-323, symbol Diode:1N4148WS
- added J7: USB_C_Receptacle, Connector_USB:USB_C_Receptacle_GCT_USB4115-03-C, symbol Connector:USB_C_Receptacle
- added NT2: Tie, NetTie:NetTie-2_SMD_Pad2.0mm, symbol Device:NetTie_2
- added R37, R47: 5,1k, Resistor_SMD:R_0603_1608Metric, symbol Device:R
- added U6: CH340C, Package_SO:SOIC-16_3.9x9.9mm_P1.27mm, symbol Interface_USB:CH340C
Connections:
- net +5V: now also C19.1, U6.16 (VCC)
- net GND: now also C19.2, C39.2, J7.A1 (GND), J7.A12 (GND), J7.B1 (GND), J7.B12 (GND), J7.S1 (SHIELD), NT2.2, R37.2, R47.2, U6.1 (GND); no longer C3.1
- net GNDPWR: now also C3.1, NT2.1
- new net: J7.A5 (CC1), R37.1
- new net: J7.A4 (VBUS), J7.A9 (VBUS), J7.B4 (VBUS), J7.B9 (VBUS)
- new net: J7.A6 (D+), J7.B6 (D+), U6.5 (UD+)
- new net: J7.A7 (D-), J7.B7 (D-), U6.6 (UD-)
- new net: J7.B5 (CC2), R47.1
- new net: C39.1, U6.4 (V3)

Commit message: hardware work
Parts:
- removed D9: 1N4148WS, Diode_SMD:D_SOD-323, symbol Diode:1N4148WS
- added R52: 5,1k, Resistor_SMD:R_0603_1608Metric, symbol Device:R
Connections:
- net +5V: now also U21.3 (~{RESET})
- net GND: now also U7.13 (~{RST})
- net UPDI: now also U6.3 (RXD), R52.1
- net at U6.2 (TXD): now also R52.2
- net DAC Reset: no longer names the net of U16.7 (PA6)
- net DAC Reset: no longer U7.13 (~{RST})
- net RESET: no longer names the net of U16.22 (PC5)
- net RESET: no longer U21.3 (~{RESET})
Other:
- moved on the sheet: TP32
Changed lines of the file:
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@@
 	(wire
 		(pts
+			(xy 80.01 128.27) (xy 115.57 128.27)
+		)
+		(stroke
+			(width 0)
+			(type default)
+		)
+	)
+	(wire
+		(pts
 			(xy 483.235 111.125) (xy 483.235 139.7)
 		)
@@
 	(wire
 		(pts
+			(xy 86.36 240.665) (xy 99.695 240.665)
+		)
+		(stroke
+			(width 0)
+			(type default)
+		)
+	)
+	(wire
+		(pts
 			(xy 486.41 92.71) (xy 486.41 95.885)
 		)
@@
 	(wire
 		(pts
+			(xy 86.36 243.205) (xy 110.49 243.205)
+		)
+		(stroke
+			(width 0)
+			(type default)
+		)
+	)
+	(wire
+		(pts
 			(xy 376.555 111.76) (xy 373.38 111.76)
 		)
@@
 	(wire
 		(pts
+			(xy 110.49 240.665) (xy 107.315 240.665)
+		)
+		(stroke
+			(width 0)
+			(type default)
+		)
+	)
+	(wire
+		(pts
 			(xy 62.23 189.23) (xy 62.23 188.595)
 		)
@@
 	(wire
 		(pts
+			(xy 110.49 243.205) (xy 110.49 240.665)
+		)
+		(stroke
+			(width 0)
+			(type default)
+		)
+	)
+	(wire
+		(pts
 			(xy 410.845 177.165) (xy 441.325 177.165)
 		)
@@
 	(wire
 		(pts
+			(xy 80.01 128.27) (xy 80.01 130.81)
+		)
+		(stroke
+			(width 0)
+			(type default)
+		)
+	)
+	(wire
+		(pts
 			(xy 408.305 92.71) (xy 428.625 92.71)
 		)
@@
 	(global_label "RESET"
 		(shape input)
-		(at 194.31 311.785 180)
+		(at 172.085 311.785 180)
 		(fields_autoplaced yes)
 		(effects
@@
 		)
 		(property "Intersheetrefs" "${INTERSHEET_REFS}"
-			(at 185.5797 311.785 0)
+			(at 163.3547 311.785 0)
 			(effects
 				(font
@@
 		)
 	)
-	(global_label "DAC Reset"
-		(shape input)
-		(at 224.79 291.465 0)
-		(fields_autoplaced yes)
-		(effects
-			(font
-				(size 1.27 1.27)
-			)
-			(justify left)
-		)
-		(property "Intersheetrefs" "${INTERSHEET_REFS}"
-			(at 237.5724 291.465 0)
-			(effects
-				(font
-					(size 1.27 1.27)
-				)
-				(justify left)
-				(hide yes)
-			)
-		)
-	)
 	(global_label "DataIn1"
 		(shape input)
@@
 	(global_label "2,5Vref"
 		(shape input)
-		(at 77.47 118.745 270)
+		(at 73.025 110.49 270)
 		(fields_autoplaced yes)
 		(effects
@@
 		)
 		(property "Intersheetrefs" "${INTERSHEET_REFS}"
-			(at 77.47 128.4431 90)
+			(at 73.025 120.1881 90)
 			(effects
 				(font
@@
 		)
 	)
-	(global_label "DAC Reset"
-		(shape input)
-		(at 115.57 128.27 180)
-		(fields_autoplaced yes)
-		(effects
-			(font
-				(size 1.27 1.27)
-			)
-			(justify right)
-		)
-		(property "Intersheetrefs" "${INTERSHEET_REFS}"
-			(at 102.7876 128.27 0)
-			(effects
-				(font
-					(size 1.27 1.27)
-				)
-				(justify right)
-				(hide yes)
-			)
-		)
-	)
 	(global_label "ISO DataOut1"
 		(shape input)
@@
 		)
 	)
+	(global_label "UPDI"
+		(shape input)
+		(at 110.49 240.665 0)
+		(fields_autoplaced yes)
+		(effects
+			(font
+				(size 1.27 1.27)
+			)
+			(justify left)
+		)
+		(property "Intersheetrefs" "${INTERSHEET_REFS}"
+			(at 117.9505 240.665 0)
+			(effects
+				(font
+					(size 1.27 1.27)
+				)
+				(justify left)
+				(hide yes)
+			)
+		)
+	)
 	(global_label "SCL"
 		(shape input)
@@
 	(symbol
 		(lib_id "Connector:TestPoint_Alt")
-		(at 77.47 118.745 0)
+		(at 73.025 110.49 0)
 		(unit 1)
 		(exclude_from_sim no)
@@
 		(fields_autoplaced yes)
 		(property "Reference" "TP32"
-			(at 80.01 114.1729 0)
+			(at 75.565 105.9179 0)
 			(effects
 				(font
@@
 		)
 		(property "Value" "Vref"
-			(at 80.01 116.7129 0)
+			(at 75.565 108.4579 0)
 			(effects
 				(font
@@
 		)
 		(property "Footprint" "TestPoint:TestPoint_Pad_D1.5mm"
-			(at 82.55 118.745 0)
+			(at 78.105 110.49 0)
 			(effects
 				(font
@@
 		)
 		(property "Datasheet" "~"
-			(at 82.55 118.745 0)
+			(at 78.105 110.49 0)
 			(effects
 				(font
@@
 		)
 		(property "Description" "test point (alternative shape)"
-			(at 77.47 118.745 0)
+			(at 73.025 110.49 0)
 			(effects
 				(font
@@
 	(symbol
 		(lib_id "power:GND")
+		(at 80.01 130.81 0)
+		(unit 1)
+		(exclude_from_sim no)
+		(in_bom yes)
+		(on_board yes)
+		(dnp no)
+		(fields_autoplaced yes)
+		(property "Reference" "#PWR0138"
+			(at 80.01 137.16 0)
+			(effects
+				(font
+					(size 1.27 1.27)
+				)
+				(hide yes)
+			)
+		)
+		(property "Value" "GND"
+			(at 80.01 135.89 0)
+			(effects
+				(font
+					(size 1.27 1.27)
+				)
+				(hide yes)
+			)
+		)
+		(property "Footprint" ""
+			(at 80.01 130.81 0)
+			(effects
+				(font
+					(size 1.27 1.27)
+				)
+				(hide yes)
+			)
+		)
+		(property "Datasheet" ""
+			(at 80.01 130.81 0)
+			(effects
+				(font
+					(size 1.27 1.27)
+				)
+				(hide yes)
+			)
+		)
+		(property "Description" ""
+			(at 80.01 130.81 0)
+			(effects
+				(font
+					(size 1.27 1.27)
+				)
+				(hide yes)
+			)
+		)
+		(pin "1"
+		)
+		(instances
+			(project "PrezisoinPowerSupply"
+				(path "/29e23d3f-5497-45d7-9b61-dc69987ec96b"
+					(reference "#PWR0138")
+					(unit 1)
+				)
+			)
+		)
+	)
+	(symbol
+		(lib_id "power:GND")
 		(at 530.225 325.12 0)
 		(unit 1)
@@
 	)
 	(symbol
-		(lib_id "Diode:1N4148WS")
-		(at 98.425 243.205 0)
+		(lib_name "+5V_1")
+		(lib_id "power:+5V")
+		(at 172.085 311.785 0)
 		(unit 1)
 		(exclude_from_sim no)
@@
 		(dnp no)
 		(fields_autoplaced yes)
-		(property "Reference" "D9"
-			(at 98.425 237.49 0)
-			(effects
-				(font
-					(size 1.27 1.27)
-				)
-			)
-		)
-		(property "Value" "1N4148WS"
-			(at 98.425 240.03 0)
-			(effects
-				(font
-					(size 1.27 1.27)
-				)
-			)
-		)
-		(property "Footprint" "Diode_SMD:D_SOD-323"
-			(at 98.425 247.65 0)
+		(property "Reference" "#PWR0139"
+			(at 172.085 315.595 0)
 			(effects
 				(font
@@
 			)
 		)
-		(property "Datasheet" "https://www.vishay.com/docs/85751/1n4148ws.pdf"
-			(at 98.425 243.205 0)
+		(property "Value" "+5V"
+			(at 172.085 306.705 0)
 			(effects
 				(font
 					(size 1.27 1.27)
 				)
-				(hide yes)
 			)
 		)
-		(property "Description" "75V 0.15A Fast switching Diode, SOD-323"
-			(at 98.425 243.205 0)
+		(property "Footprint" ""
+			(at 172.085 311.785 0)
 			(effects
 				(font
@@
 			)
 		)
-		(property "Sim.Device" "D"
-			(at 98.425 243.205 0)
+		(property "Datasheet" ""
+			(at 172.085 311.785 0)
 			(effects
 				(font
@@
 			)
 		)
-		(property "Sim.Pins" "1=K 2=A"
-			(at 98.425 243.205 0)
+		(property "Description" "Power symbol creates a global label with name \"+5V\""
+			(at 172.085 311.785 0)
 			(effects
 				(font
@@
 			)
 		)
-		(pin "2"
-		)
 		(pin "1"
 		)
 		(instances
-			(project ""
+			(project "PrezisoinPowerSupply"
 				(path "/29e23d3f-5497-45d7-9b61-dc69987ec96b"
-					(reference "D9")
+					(reference "#PWR0139")
 					(unit 1)
 				)
@@
 					(unit 1)
 				)
+			)
+		)
+	)
+	(symbol
+		(lib_id "Device:R")
+		(at 103.505 240.665 270)
+		(unit 1)
+		(exclude_from_sim no)
+		(in_bom yes)
+		(on_board yes)
+		(dnp no)
+		(property "Reference" "R52"
+			(at 103.505 238.76 90)
+			(effects
+				(font
+					(size 1.27 1.27)
+				)
+			)
+		)
+		(property "Value" "5,1k"
+			(at 103.505 242.57 90)
+			(effects
+				(font
+					(size 1.27 1.27)
+				)
+			)
+		)
+		(property "Footprint" "Resistor_SMD:R_0603_1608Metric"
+			(at 103.505 238.887 90)
+			(effects
+				(font
+					(size 1.27 1.27)
+				)
+				(hide yes)
+			)
+		)
+		(property "Datasheet" "~"
+			(at 103.505 240.665 0)
+			(effects
+				(font
+					(size 1.27 1.27)
+				)
+				(hide yes)
+			)
+		)
+		(property "Description" ""
+			(at 103.505 240.665 0)
+			(effects
+				(font
+					(size 1.27 1.27)
+				)
+				(hide yes)
+			)
+		)
+		(pin "1"
+		)
+		(pin "2"
+		)
+		(instances
+			(project "PrezisoinPowerSupply"
+				(path "/29e23d3f-5497-45d7-9b61-dc69987ec96b"
+					(reference "R52")
+					(unit 1)
+				)

Commit message: hardware work ##
Parts:
- added D9: LED, LED_SMD:LED_0603_1608Metric, symbol Device:LED
- added K2: G2RL-2, Relay_THT:Relay_SPDT_Omron_G2RL-1-E, symbol Relay:G2RL-2
- added R53, R54: 1k, Resistor_SMD:R_0603_1608Metric, symbol Device:R
Connections:
- net +5V: now also R53.1
- net 2,5Vref: now also R54.1; no longer C48.1, U21.9 (REFP)
- net GND: now also D9.1 (K)
- new net: D9.2 (A), R53.2
- new net: C48.1, R54.2, U21.9 (REFP)

Commit message: hardware relay
Parts:
- removed K2: G2RL-2, Relay_THT:Relay_SPDT_Omron_G2RL-1-E, symbol Relay:G2RL-2
- added K3: SANYOU_SRD_Form_C, Relay_THT:Relay_SPDT_SANYOU_SRD_Series_Form_C, symbol Relay:SANYOU_SRD_Form_C
- added R55: 0.05, Library:R 2728 4Wire, symbol Device:R_Shunt
Connections:
- net outLOW: now also K3.1; no longer R51.1
- new net: K3.4, R51.1
Other:
- moved on the sheet: D8, F2, J6, R51

Commit message: range switch
Parts:
- removed J4: LEDs, Connector_JST:JST_XH_B3B-XH-A_1x03_P2.50mm_Vertical, symbol Connector:Conn_01x03_Pin
- removed J5: Sense, Connector_JST:JST_XH_B4B-XH-A_1x04_P2.50mm_Vertical, symbol Connector:Conn_01x04_Pin
- removed R55: 0.05, Library:R 2728 4Wire, symbol Device:R_Shunt
- added C42, C49, C50: 100n, Capacitor_SMD:C_0603_1608Metric, symbol Device:C
- added D10: 1N4007, Diode_SMD:D_SOD-123F, symbol Device:D
- added J8: Conn_01x08_Socket, Connector_JST:JST_GH_BM08B-GHS-TBT_1x08-1MP_P1.25mm_Vertical, symbol Connector:Conn_01x08_Socket
- added Q3: MMBT3904, Package_TO_SOT_SMD:SOT-23-3, symbol Transistor_BJT:MMBT3904
- added R55, R56: 10 0,05%, Resistor_SMD:R_0603_1608Metric, symbol Device:R
- added R57: 1k, Resistor_SMD:R_0603_1608Metric, symbol Device:R
- added U15: OPA2192, Package_SO:SOIC-8_3.9x4.9mm_P1.27mm, symbol Device:Opamp_Dual
- added U17: TS5A23159RSE, Package_DFN_QFN:Texas_R-PUQFN-N10, symbol Analog_Switch:TS5A23159RSE
Connections:
- net +12V: now also K3.2, C50.1, D10.1 (K)
- net +5V: now also C49.1, J8.7 (Pin_7), U17.8 (VCC)
- net +VDC: now also C42.1, U15.8 (V+)
- net -12V: no longer D3.1 (K), D4.1 (K)
- net ExSense+: now also J8.1 (Pin_1); no longer R5.1
- net ExSense-: now also J8.2 (Pin_2); no longer R6.1
- net GND: now also D3.1 (K), D4.1 (K), C42.2, C49.2, C50.2, J8.5 (Pin_5), Q3.2 (E), U15.4 (V-), U17.3 (GND)
- net GNDPWR: now also R55.1, R56.1, U17.2
- net IntSense+: now also J8.3 (Pin_3); no longer R5.2
- net IntSense-: now also J8.4 (Pin_4); no longer R6.2
- net LED_ON: now also J8.6 (Pin_6)
- net LED_SenseEx: now also J8.8 (Pin_8)
- net outHi: now also R5.1
- net outLOW: now also R6.1
- net at D3.3 (K), F3.1: now also U15.3 (+); no longer R21.2
- net at F3.2, K1.9: now also R5.2
- net at F4.2, K1.4: now also R6.2
- net at R41.2: now also U17.6; no longer R51.2
- net at D4.3 (K), F4.1: now also U15.5 (+); no longer R22.2
- net at R39.2: now also U17.10; no longer R51.3
- net at K3.3: now also R55.2, R56.2, U17.4
- net at K3.5: now also D10.2 (A), Q3.3 (C)
- new net: R51.2, U17.7
- new net: Q3.1 (B), R57.2
- new net: R22.2, U15.6 (-), U15.7
- new net: R21.2, U15.1, U15.2 (-)
- new net: R51.3, U17.9
- new net RangeSW: R57.1, U17.1, U17.5
Other:
- moved on the sheet: C35, D2, D3, D4, F3, F4, K1, Q6, Q7, Q8, R38, R49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
