File: Hardware/Modul/PrezisoinPowerSupply 2_3/buckLDO.kicad_sch (KiCad schematic)
At the start: 35 parts, among them U1 AP63200WU, U13 TME-1212S, U14 LM7805_TO220, U18 LM7812_TO220, U20 ICM7555xB

Commit message: new revision
Parts:
- added U23: TEN 3-2422, Library:Traco TEN 3-2422, symbol SymbolLibary:TEN_3-2422
Connections:
- net Vin: now also U23.22 (Vin), U23.23 (Vin)
- new net: U23.16 (Common), U23.9 (Common)
- new net -Vin: U23.2 (-Vin), U23.3 (-Vin)
Changed lines of the file:
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@@
+	)
+	(symbol
+		(lib_id "SymbolLibary:TEN_3-2422")
+		(at 129.54 44.45 0)
+		(unit 1)
+		(exclude_from_sim no)
+		(in_bom yes)
+		(on_board yes)
+		(dnp no)
+		(fields_autoplaced yes)
+		(property "Reference" "U23"
+			(at 129.54 35.56 0)
+			(effects
+				(font
+					(size 1.27 1.27)
+				)
+			)
+		)
+		(property "Value" "TEN 3-2422"
+			(at 129.54 38.1 0)
+			(effects
+				(font
+					(size 1.27 1.27)
+				)
+			)
+		)
+		(property "Footprint" "Library:Traco TEN 3-2422"
+			(at 129.54 44.45 0)
+			(effects
+				(font
+					(size 1.27 1.27)
+				)
+				(hide yes)
+			)
+		)
+		(property "Datasheet" ""
+			(at 129.54 44.45 0)
+			(effects
+				(font
+					(size 1.27 1.27)
+				)
+				(hide yes)
+			)
+		)
+		(property "Description" ""
+			(at 129.54 44.45 0)
+			(effects
+				(font
+					(size 1.27 1.27)
+				)
+				(hide yes)
+			)
+		)
+		(pin "16"
+		)
+		(pin "23"
+		)
+		(pin "3"
+		)
+		(pin "9"
+		)
+		(pin "11"
+		)
+		(pin "14"
+		)
+		(pin "2"
+		)
+		(pin "22"
+		)
+		(instances
+			(project ""
+				(path "/29e23d3f-5497-45d7-9b61-dc69987ec96b/adc78fce-9a4a-4340-b242-c3940e74dfc2"
+					(reference "U23")
+					(unit 1)
+				)
+			)
+		)
 	)
 	(symbol
