File: Hardware/Modul/PrezisoinPowerSupply 2_4/PrezisoinPowerSupply.kicad_pcb (KiCad board)
At the start: 4 copper layers, 91 x 100 mm, 232 parts, among them J1 Supply, J2 Conn_01x03_Pin, J3 Conn_02x05_Odd_Even, J4 Conn_01x10_Socket, J6 Output, J7 USB_C_Receptacle, K1 EE2-5NU, Q1 IRFP240, Q10 DMN2008, Q2 IRFP9240, Q3 DMN2008, Q4 IRFP9240, Q5 MMBT3904, Q6 MMBT3904, Q7 MMBT3904, Q8 MMBT3904, Q9 IRFP240, U1 AP63200WU, U10 OPA4189, U11 OPA4189, U12 OPA189, U13 TME-1212S, U14 LM7805_TO220, U15 OPA2192, U16 ATtiny3227-M, U17 TS5A23159RSE, U18 LM7812_TO220, U19 TLV9301xDBV, U2 DG469, U20 ICM7555xB, U21 ADS1219, U22 SN74LVC1G14DBV, U23 TEN 3-2422, U3 ADA4522, U4 CPC1017N, U5 ISO7763FDBQ, U6 CH340C, U7 DAC8564C/D, U8 MCP9700Ax-ETT, U9 MCP9700Ax-ETT

Commit message: new revision
Parts:
- removed C13, C17, C21, C22, C25, C26, C27, C28: 10u, Capacitor_SMD:C_1206_3216Metric
- removed C14: 100n, Capacitor_SMD:C_1206_3216Metric
- removed C19, C23, C39, C50: 100n, Capacitor_SMD:C_0603_1608Metric
- removed C24: 56p-100p, Capacitor_SMD:C_0603_1608Metric
- removed J7: USB_C_Receptacle, Connector_USB:USB_C_Receptacle_GCT_USB4115-03-C
- removed JP2: USB PW Link, Jumper:SolderJumper-2_P1.3mm_Open_RoundedPad1.0x1.5mm
- removed L1: 10u, Inductor_SMD:L_Taiyo-Yuden_NR-80xx
- removed R29: 200k, Resistor_SMD:R_0603_1608Metric
- removed R30: 12k, Resistor_SMD:R_0603_1608Metric
- removed R37, R47, R52: 5,1k, Resistor_SMD:R_0603_1608Metric
- removed R57: 100, Resistor_SMD:R_0603_1608Metric
- removed U1: AP63200WU, Package_TO_SOT_SMD:TSOT-23-6
- removed U13: TME-1212S, Converter_DCDC:Converter_DCDC_TRACO_TME_03xxS_05xxS_12xxS_Single_THT
- removed U18: LM7812_TO220, Package_TO_SOT_THT:TO-220-3_Vertical
- removed U6: CH340C, Package_SO:SOIC-16_3.9x9.9mm_P1.27mm
- C15, C4: value 100n -> 1u; footprint Capacitor_SMD:C_0603_1608Metric -> Capacitor_SMD:C_1206_3216Metric
- C16: value 10u -> 1u
- U8, U9: value MCP9700Ax-ETT -> MCP9700
- moved C15 68.0 mm to (122.6, 34.1), turned to 0 degrees
- moved C4 67.2 mm to (122.6, 30.8), turned to 0 degrees
- moved C16 64.6 mm to (122.6, 37.5), turned to 0 degrees
- moved C34 40.9 mm to (190.3, 42.0)
- moved C52 40.9 mm to (205.4, 47.5)
- moved C53 40.9 mm to (203.7, 47.5)
- moved C54 40.9 mm to (194.8, 41.5)
- moved C55 40.9 mm to (193.3, 48.4)
- moved D6 40.9 mm to (193.3, 44.9)
- moved U20 40.9 mm to (202.8, 43.1)
- moved C37 40.9 mm to (208.2, 41.1)
- moved C51 40.9 mm to (208.2, 42.7)
- moved R31 40.9 mm to (198.1, 41.2)
- moved R48 40.9 mm to (197.3, 43.6)
- moved C18 40.9 mm to (196.2, 50.9)
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Connections:
- C15 pad 2: /buckConLDO/-12V -> /buckConLDO/12V
- C16 pad 1: GND -> -12V
- C16 pad 2: /buckConLDO/-12V -> GND
- C29 pad 2: GND -> Net-(U14-GND)
- C30 pad 2: GND -> Net-(U14-GND)
- C4 pad 1: /buckConLDO/12V -> GND
- C4 pad 2: GND -> +VDC
- JP5 pad 1: /buckConLDO/-12V -> /-12V
- TP6 pad 1: /buckConLDO/-12V -> /-12V
- U14 pad 2: GND -> Net-(U14-GND)
- U23 pad 11: unconnected-(U23--Vout-Pad11) -> -12V
- U23 pad 14: unconnected-(U23-+Vout-Pad14) -> /buckConLDO/12V
- U23 pad 16: Net-(U23-Common-Pad16) -> GND
- U23 pad 2: -Vin -> GND
- U23 pad 3: -Vin -> GND
- U23 pad 9: Net-(U23-Common-Pad16) -> GND
Routing:
- net +VDC: track 164.5 -> 107.6 mm
- net /buckConLDO/+15V: track 50.0 -> 0.00 mm, vias 2 -> 0
- net /buckConLDO/12V: track 95.3 -> 59.0 mm
- net /buckConLDO/-12V: track 22.1 -> 0.00 mm
- net Net-(U1-FB): track 5.35 -> 0.00 mm
- net /-12V: track 0.00 -> 3.15 mm
- net /buckConLDO/..36V: track 24.6 -> 27.4 mm
- net /outHi: track 185.9 -> 188.3 mm
- net Net-(U1-BST): track 1.57 -> 0.00 mm
- net /buckConLDO/SW: track 1.56 -> 0.00 mm
- net GND: vias 148 -> 109
- removed copper zone on F.Cu, net +VDC
- removed copper zone on F.Cu, net /buckConLDO/+15V
- removed copper zone on F.Cu, net /buckConLDO/SW

Commit message: heatsink
Parts:
- removed the REF** at (167.0, 100.0)
- removed the REF** at (125.0, 100.0)
- added R29: 0.1, Resistor_THT:R_Bare_Metal_Element_L21.3mm_W4.8mm_P20.30mm, B.Cu at (133.9, 97.5)
- added R30: 0.1, Resistor_THT:R_Bare_Metal_Element_L21.3mm_W4.8mm_P20.30mm, B.Cu at (133.9, 103.8)
- added R37: 0.1, Resistor_THT:R_Bare_Metal_Element_L21.3mm_W4.8mm_P20.30mm, B.Cu at (237.4, 187.8)
- added R47: 0.1, Resistor_THT:R_Bare_Metal_Element_L21.3mm_W4.8mm_P20.30mm, B.Cu at (231.9, 187.8)
- added REF**: 78350 Heatsink, Library:78350 Heatsink, B.Cu at (222.8, 200.0)
- added REF**: 78350 Heatsink, Library:78350 Heatsink, B.Cu at (159.2, 50.0)
- R16, R17, R18, R7: value 0.05 -> 0.1; footprint Resistor_SMD:R_2512_6332Metric -> Resistor_THT:R_Bare_Metal_Element_L21.3mm_W4.8mm_P20.30mm; moved to B.Cu
- moved R17 154.4 mm to (262.1, 133.1), turned to 180 degrees
- moved C4 122.3 mm to (210.6, 115.6)
- moved C15 111.2 mm to (210.0, 102.8), turned to 180 degrees
- moved JP7 98.2 mm to (288.3, 106.4)
- moved C53 98.2 mm to (284.4, 103.6)
- moved R31 98.2 mm to (278.7, 97.3)
- moved C18 98.2 mm to (276.9, 106.9)
- moved C34 98.2 mm to (271.0, 98.1)
- moved C37 98.2 mm to (288.8, 97.2)
- moved C51 98.2 mm to (288.8, 98.8)
- moved C52 98.2 mm to (286.1, 103.6)
- moved C54 98.2 mm to (275.5, 97.6)
- moved C55 98.2 mm to (274.0, 104.5)
- moved D6 98.2 mm to (274.0, 101.0)
- moved JP6 98.2 mm to (289.2, 101.4)
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Connections:
- R17 pad 1: /outHi -> Net-(Q1-S)
- R17 pad 2: Net-(Q4-S) -> /outHi
- R18 pad 2: Net-(Q2-S) -> Net-(Q4-S)
Routing:
- net /buckConLDO/12V: track 59.0 -> 0.00 mm
- net /outHi: track 188.3 -> 145.3 mm, vias 27 -> 11
- net GNDPWR: track 169.3 -> 132.7 mm
- net (no net): track 0.00 -> 29.4 mm
- net Net-(JP2-A): track 23.4 -> 0.00 mm, vias 5 -> 0
- net /buckConLDO/Vout 5V: track 16.8 -> 2.62 mm
- net Net-(U6-TXD): track 11.1 -> 0.00 mm
- net Net-(FB6-Pad1): track 117.7 -> 107.3 mm
- net Net-(J7-CC2): track 8.77 -> 0.00 mm, vias 2 -> 0
- net GND: track 94.5 -> 85.8 mm, vias 109 -> 103
- net Net-(U6-RXD): track 8.04 -> 0.00 mm
- net Net-(U6-UD-): track 7.61 -> 0.00 mm, vias 2 -> 0
- net Net-(U6-UD+): track 6.98 -> 0.00 mm
- net Net-(U6-V3): track 6.79 -> 0.00 mm
- net Net-(Q2-G): track 4.91 -> 0.41 mm
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Other:
- board size 91 x 100 mm -> 100 x 150 mm
