File: Hardware/Modul/PrezisoinPowerSupply 2_4/buckLDO.kicad_sch (KiCad schematic)
At the start: 21 parts, among them U14 LM7805_TO220, U20 ICM7555xB, U23 TEN 3-2422

Commit message: new front dist and updates
Changed lines of the file:
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@@
 (kicad_sch
-	(version 20231120)
+	(version 20250114)
 	(generator "eeschema")
-	(generator_version "8.0")
+	(generator_version "9.0")
 	(paper "A4")
 	(junction
@@
 	(label "..36V"
 		(at 184.15 127 0)
-		(fields_autoplaced yes)
 		(effects
 			(font
@@
 	(label "12V"
 		(at 99.695 117.475 0)
-		(fields_autoplaced yes)
 		(effects
 			(font
@@
 	(label "Vin"
 		(at 189.23 144.78 0)
-		(fields_autoplaced yes)
 		(effects
 			(font
@@
 	(label "..24V"
 		(at 181.61 144.78 0)
-		(fields_autoplaced yes)
 		(effects
 			(font
@@
 	(label "+15V"
 		(at 85.725 117.475 0)
-		(fields_autoplaced yes)
 		(effects
 			(font
@@
 	(label "12V"
 		(at 133.985 71.12 0)
-		(fields_autoplaced yes)
 		(effects
 			(font
@@
 		(shape input)
 		(at 165.1 71.12 90)
-		(fields_autoplaced yes)
 		(effects
 			(font
@@
 		(shape input)
 		(at 128.27 71.12 90)
-		(fields_autoplaced yes)
 		(effects
 			(font
@@
 		(shape input)
 		(at 113.03 162.56 90)
-		(fields_autoplaced yes)
 		(effects
 			(font
@@
 		(shape input)
 		(at 193.675 127 0)
-		(fields_autoplaced yes)
-		(effects
-			(font
+		(effects
+			(font
