File: Hardware/Modul/PrezisoinPowerSupply 2_4/PrezisoinPowerSupply.kicad_sch (KiCad schematic)
At the start: 174 parts, among them J1 Supply, J2 Conn_01x03_Pin, J3 Conn_02x05_Odd_Even, J4 Conn_01x10_Socket, J6 Output, K1 EE2-5NU, Q1 IRFP240, Q10 DMN2008, Q2 IRFP9240, Q3 DMN2008, Q4 IRFP9240, Q5 MMBT3904, Q6 MMBT3904, Q7 MMBT3904, Q8 MMBT3904, Q9 IRFP240, U10 OPA4189, U11 OPA4189, U12 OPA189, U15 OPA2192, U16 ATtiny3227-M, U17 TS5A23159RSE, U19 TLV9301xDBV, U2 DG469, U21 ADS1219, U22 SN74LVC1G14DBV, U3 ADA4522, U4 CPC1017N, U5 ISO7763FDBQ, U7 DAC8564C/D, U8 MCP9700, U9 MCP9700

Commit message: heatsink
Parts:
- added R29, R30, R37, R47: 0.1, Resistor_THT:R_Bare_Metal_Element_L21.3mm_W4.8mm_P20.30mm, symbol Device:R
- R16, R17, R18, R7: value 0.05 -> 0.1; footprint Resistor_SMD:R_2512_6332Metric -> Resistor_THT:R_Bare_Metal_Element_L21.3mm_W4.8mm_P20.30mm
Connections:
- net RangeSW: no longer R41.2, U17.6
- net outHi: now also R17.2, R29.2, R30.1, R37.1, R47.1; no longer R17.1
- net at Q1.3 (S), R16.1: now also R17.1
- net at Q9.3 (S), R7.1: now also R29.1
- net at Q4.3 (S): now also R18.2, R30.2; no longer R17.2
- net at Q2.3 (S): now also R37.2, R47.2; no longer R18.2
- new net: R41.2, U17.6
Other:
- moved on the sheet: C1, C10, C11, C12, C2, C3, C31, C32, C33, C35, C36, C38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

Commit message: ??
Other:
- added sheet MCU&ISO (MCU&ISO.kicad_sch)
- moved on the sheet: C40, C43, C44, C46, C47, D9, FB1, J2, J3, R53, TP1, TP12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
